File: sc_v1.brd (EAGLE design)
At the start: 30.8 x 15.1 mm, 20 parts, among them IC1 CP2102, J1 TYPE-C-31-M-12, U2 3.3V

Commit message: Add files via upload
Parts:
- moved IC1 0.80 mm to (12.7, 2.75)
Connections:
- removed net N$5: C1.2, IC1.6
- net +3V3: now also C1.2, IC1.6, IC1.7
- net +5V: no longer IC1.7
Routing:
- net +3V3: track 22.7 -> 30.0 mm, vias 2 -> 3
- net N$5: track 1.84 -> 0.00 mm
- net TMS: track 15.4 -> 16.5 mm
- net TCK: track 14.1 -> 15.2 mm
- net PB01: track 21.0 -> 21.8 mm
- net PB00: track 20.2 -> 21.0 mm
- net N$1: track 5.42 -> 6.22 mm
- net TX: track 6.87 -> 7.67 mm
- net RX: track 14.0 -> 14.8 mm
- net N$3: track 2.14 -> 1.34 mm
- net N$2: track 8.22 -> 8.81 mm
- net GND: track 8.22 -> 8.04 mm, vias 24 -> 28

Commit message: Add files via upload
Parts:
- moved R2 1.00 mm to (9.10, 3.02), turned to 90 degrees
Connections:
- net +3V3: now also R2.1
- net +5V: no longer R2.1
Routing:
- net +3V3: track 30.0 -> 34.3 mm, vias 3 -> 4
- net TCK: track 15.2 -> 16.4 mm
- net TMS: track 16.5 -> 17.7 mm
- net TDI: track 21.7 -> 21.2 mm
- net GND: vias 28 -> 29

Commit message: Add files via upload
Parts:
- added C2: 100n, discretes-dev:CAPC1005X40N
- moved R1 0.50 mm to (3.74, 8.64)
- moved R5 0.50 mm to (3.75, 6.12)
Connections:
- net +3V3: now also C2.1
- net GND: now also C2.2
Routing:
- net +3V3: track 34.3 -> 36.8 mm, vias 4 -> 5
- net N$4: track 3.63 -> 3.13 mm
- net GND: vias 29 -> 28
Other:
- board text added: "."

Commit message: Add files via upload
Parts:
- added R6, R7, R8: 10k, SparkFun-Resistors:0402
- moved R2 0.95 mm to (9.01, 3.96)
- moved D4 0.30 mm to (10.3, 7.78)
Connections:
- new net N$5: IC1.11, R6.2
- net GND: now also R6.1, R7.2, R8.2
- net PB00: now also R7.1
- net PB01: now also R8.1
Routing:
- net N$5: track 0.00 -> 2.32 mm, vias 0 -> 1
- net PB01: track 21.8 -> 22.8 mm, vias 0 -> 1
- net +3V3: track 36.8 -> 37.8 mm
- net PB00: track 21.4 -> 22.3 mm, vias 0 -> 1
- net GND: vias 28 -> 25
