File: sc_v1.sch (EAGLE design)
At the start: 20 parts, among them IC1 CP2102, J1 TYPE-C-31-M-12, U2 3.3V

Commit message: Add files via upload
Connections:
- removed net N$5: C1.2, IC1.VDD
- net +3V3: now also C1.2, IC1.REGIN, IC1.VDD
- net +5V: no longer IC1.REGIN
Other:
- moved on the sheet: C1, TP1, TP2, TP3, TP4, TP5, TP6, TP7
Changed lines of the file:
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@@
 <part name="TP7" library="testpad" library_urn="urn:adsk.eagle:library:385" deviceset="PTR1" device="TP10R" package3d_urn="urn:adsk.eagle:package:27959/1"/>
 <part name="C1" library="discretes-dev" deviceset="CAP0402" device="" value="100nf"/>
+<part name="+3V1" library="supply1" library_urn="urn:adsk.eagle:library:371" deviceset="+3V3" device=""/>
 </parts>
 <sheets>
@@
 <attribute name="VALUE" x="20.32" y="104.14" size="1.778" layer="96" rot="R180"/>
 </instance>
-<instance part="P+2" gate="1" x="22.86" y="60.96" smashed="yes">
-<attribute name="VALUE" x="20.32" y="55.88" size="1.778" layer="96" rot="R90"/>
+<instance part="P+2" gate="1" x="17.78" y="50.8" smashed="yes" rot="R90">
+<attribute name="VALUE" x="22.86" y="48.26" size="1.778" layer="96" rot="R180"/>
 </instance>
 <instance part="P+3" gate="1" x="78.74" y="53.34" smashed="yes" rot="R270">
 <attribute name="VALUE" x="73.66" y="55.88" size="1.778" layer="96"/>
 </instance>
-<instance part="GND5" gate="1" x="15.24" y="58.42" smashed="yes" rot="R180">
-<attribute name="VALUE" x="17.78" y="60.96" size="1.778" layer="96" rot="R180"/>
+<instance part="GND5" gate="1" x="2.54" y="45.72" smashed="yes" rot="R270">
+<attribute name="VALUE" x="0" y="48.26" size="1.778" layer="96" rot="R270"/>
 </instance>
 <instance part="U2" gate="G$1" x="137.16" y="88.9" smashed="yes">
@@
 <attribute name="VALUE" x="63.5" y="60.96" size="1.778" layer="96"/>
 </instance>
-<instance part="TP1" gate="G$1" x="182.88" y="53.34" smashed="yes" rot="R90">
-<attribute name="NAME" x="189.23" y="52.324" size="1.778" layer="95"/>
-<attribute name="TP_SIGNAL_NAME" x="185.42" y="54.61" size="1.778" layer="97" rot="R90"/>
-</instance>
-<instance part="TP2" gate="G$1" x="182.88" y="50.8" smashed="yes" rot="R90">
-<attribute name="NAME" x="189.23" y="49.784" size="1.778" layer="95"/>
-<attribute name="TP_SIGNAL_NAME" x="185.42" y="52.07" size="1.778" layer="97" rot="R90"/>
-</instance>
-<instance part="TP3" gate="G$1" x="182.88" y="48.26" smashed="yes" rot="R90">
-<attribute name="NAME" x="189.23" y="47.244" size="1.778" layer="95"/>
-<attribute name="TP_SIGNAL_NAME" x="185.42" y="49.53" size="1.778" layer="97" rot="R90"/>
-</instance>
-<instance part="TP4" gate="G$1" x="182.88" y="45.72" smashed="yes" rot="R90">
-<attribute name="NAME" x="189.23" y="44.704" size="1.778" layer="95"/>
-<attribute name="TP_SIGNAL_NAME" x="185.42" y="46.99" size="1.778" layer="97" rot="R90"/>
-</instance>
-<instance part="TP5" gate="G$1" x="182.88" y="43.18" smashed="yes" rot="R90">
-<attribute name="NAME" x="189.23" y="42.164" size="1.778" layer="95"/>
-<attribute name="TP_SIGNAL_NAME" x="185.42" y="44.45" size="1.778" layer="97" rot="R90"/>
-</instance>
-<instance part="TP6" gate="G$1" x="182.88" y="40.64" smashed="yes" rot="R90">
-<attribute name="NAME" x="189.23" y="39.624" size="1.778" layer="95"/>
-<attribute name="TP_SIGNAL_NAME" x="185.42" y="41.91" size="1.778" layer="97" rot="R90"/>
-</instance>
-<instance part="TP7" gate="G$1" x="182.88" y="38.1" smashed="yes" rot="R90">
-<attribute name="NAME" x="189.23" y="37.084" size="1.778" layer="95"/>
-<attribute name="TP_SIGNAL_NAME" x="185.42" y="39.37" size="1.778" layer="97" rot="R90"/>
-</instance>
-<instance part="C1" gate="G$1" x="15.24" y="50.8" smashed="yes">
-<attribute name="NAME" x="16.764" y="52.451" size="1.778" layer="95" font="vector"/>
+<instance part="TP1" gate="G$1" x="99.06" y="48.26" smashed="yes" rot="R90">
+<attribute name="NAME" x="105.41" y="47.244" size="1.778" layer="95"/>
+<attribute name="TP_SIGNAL_NAME" x="101.6" y="49.53" size="1.778" layer="97" rot="R90"/>
+</instance>
+<instance part="TP2" gate="G$1" x="99.06" y="45.72" smashed="yes" rot="R90">
+<attribute name="NAME" x="105.41" y="44.704" size="1.778" layer="95"/>
+<attribute name="TP_SIGNAL_NAME" x="101.6" y="46.99" size="1.778" layer="97" rot="R90"/>
+</instance>
+<instance part="TP3" gate="G$1" x="99.06" y="43.18" smashed="yes" rot="R90">
+<attribute name="NAME" x="105.41" y="42.164" size="1.778" layer="95"/>
+<attribute name="TP_SIGNAL_NAME" x="101.6" y="44.45" size="1.778" layer="97" rot="R90"/>
+</instance>
+<instance part="TP4" gate="G$1" x="99.06" y="40.64" smashed="yes" rot="R90">
+<attribute name="NAME" x="105.41" y="39.624" size="1.778" layer="95"/>
+<attribute name="TP_SIGNAL_NAME" x="101.6" y="41.91" size="1.778" layer="97" rot="R90"/>
+</instance>
+<instance part="TP5" gate="G$1" x="99.06" y="38.1" smashed="yes" rot="R90">
+<attribute name="NAME" x="105.41" y="37.084" size="1.778" layer="95"/>
+<attribute name="TP_SIGNAL_NAME" x="101.6" y="39.37" size="1.778" layer="97" rot="R90"/>
+</instance>
+<instance part="TP6" gate="G$1" x="99.06" y="35.56" smashed="yes" rot="R90">
+<attribute name="NAME" x="105.41" y="34.544" size="1.778" layer="95"/>
+<attribute name="TP_SIGNAL_NAME" x="101.6" y="36.83" size="1.778" layer="97" rot="R90"/>
+</instance>
+<instance part="TP7" gate="G$1" x="99.06" y="33.02" smashed="yes" rot="R90">
+<attribute name="NAME" x="105.41" y="32.004" size="1.778" layer="95"/>
+<attribute name="TP_SIGNAL_NAME" x="101.6" y="34.29" size="1.778" layer="97" rot="R90"/>
+</instance>
+<instance part="C1" gate="G$1" x="10.16" y="45.72" smashed="yes" rot="R90">
+<attribute name="NAME" x="5.969" y="47.244" size="1.778" layer="95" font="vector"/>
+</instance>
+<instance part="+3V1" gate="G$1" x="15.24" y="60.96" smashed="yes">
+<attribute name="VALUE" x="12.7" y="55.88" size="1.778" layer="96" rot="R90"/>
 </instance>
 </instances>
@@
 <segment>
 <pinref part="TP1" gate="G$1" pin="TP"/>
-<wire x1="180.34" y1="53.34" x2="172.72" y2="53.34" width="0.1524" layer="91"/>
-<label x="172.72" y="53.34" size="1.778" layer="95"/>
-</segment>
-<segment>
+<wire x1="96.52" y1="48.26" x2="88.9" y2="48.26" width="0.1524" layer="91"/>
+<label x="88.9" y="48.26" size="1.778" layer="95"/>
+</segment>
+<segment>
+<pinref part="C1" gate="G$1" pin="1"/>
+<wire x1="6.35" y1="45.72" x2="5.08" y2="45.72" width="0.1524" layer="91"/>
 <pinref part="GND5" gate="1" pin="GND"/>
-<pinref part="C1" gate="G$1" pin="1"/>
-<wire x1="15.24" y1="55.88" x2="15.24" y2="54.61" width="0.1524" layer="91"/>
 </segment>
 </net>
@@
 </segment>
 <segment>
-<pinref part="IC1" gate="G$1" pin="VBUS"/>
-<pinref part="IC1" gate="G$1" pin="REGIN"/>
-<wire x1="22.86" y1="50.8" x2="22.86" y2="53.34" width="0.1524" layer="91"/>
-<wire x1="22.86" y1="53.34" x2="22.86" y2="58.42" width="0.1524" layer="91"/>
-<junction x="22.86" y="53.34"/>
-<pinref part="P+2" gate="1" pin="+5V"/>
-</segment>
-<segment>
 <pinref part="P+3" gate="1" pin="+5V"/>
 <wire x1="73.66" y1="53.34" x2="76.2" y2="53.34" width="0.1524" layer="91"/>
 <pinref part="R2" gate="G$1" pin="1"/>
+</segment>
+<segment>
+<pinref part="P+2" gate="1" pin="+5V"/>
+<pinref part="IC1" gate="G$1" pin="VBUS"/>
+<wire x1="20.32" y1="50.8" x2="22.86" y2="50.8" width="0.1524" layer="91"/>
 </segment>
 </net>
@@
 <segment>
 <pinref part="TP2" gate="G$1" pin="TP"/>
-<wire x1="180.34" y1="50.8" x2="172.72" y2="50.8" width="0.1524" layer="91"/>
-<label x="172.72" y="50.8" size="1.778" layer="95"/>
+<wire x1="96.52" y1="45.72" x2="88.9" y2="45.72" width="0.1524" layer="91"/>
+<label x="88.9" y="45.72" size="1.778" layer="95"/>
+</segment>
+<segment>
+<pinref part="IC1" gate="G$1" pin="VDD"/>
+<pinref part="C1" gate="G$1" pin="2"/>
+<wire x1="13.97" y1="45.72" x2="15.24" y2="45.72" width="0.1524" layer="91"/>
+<pinref part="+3V1" gate="G$1" pin="+3V3"/>
+<wire x1="15.24" y1="45.72" x2="22.86" y2="45.72" width="0.1524" layer="91"/>
+<wire x1="15.24" y1="58.42" x2="15.24" y2="53.34" width="0.1524" layer="91"/>
+<junction x="15.24" y="45.72"/>
+<pinref part="IC1" gate="G$1" pin="REGIN"/>
+<wire x1="15.24" y1="53.34" x2="15.24" y2="45.72" width="0.1524" layer="91"/>
+<wire x1="22.86" y1="53.34" x2="15.24" y2="53.34" width="0.1524" layer="91"/>
+<junction x="15.24" y="53.34"/>
 </segment>
 </net>
@@
 <segment>
 <pinref part="TP6" gate="G$1" pin="TP"/>
-<wire x1="180.34" y1="40.64" x2="172.72" y2="40.64" width="0.1524" layer="91"/>
-<label x="172.72" y="40.64" size="1.778" layer="95"/>
+<wire x1="96.52" y1="35.56" x2="88.9" y2="35.56" width="0.1524" layer="91"/>
+<label x="88.9" y="35.56" size="1.778" layer="95"/>
 </segment>
 </net>
@@
 <segment>
 <pinref part="TP7" gate="G$1" pin="TP"/>
-<wire x1="180.34" y1="38.1" x2="172.72" y2="38.1" width="0.1524" layer="91"/>
-<label x="172.72" y="38.1" size="1.778" layer="95"/>
+<wire x1="96.52" y1="33.02" x2="88.9" y2="33.02" width="0.1524" layer="91"/>
+<label x="88.9" y="33.02" size="1.778" layer="95"/>
 </segment>
 </net>
@@
 <segment>
 <pinref part="TP5" gate="G$1" pin="TP"/>
-<wire x1="180.34" y1="43.18" x2="172.72" y2="43.18" width="0.1524" layer="91"/>
-<label x="172.72" y="43.18" size="1.778" layer="95"/>
+<wire x1="96.52" y1="38.1" x2="88.9" y2="38.1" width="0.1524" layer="91"/>
+<label x="88.9" y="38.1" size="1.778" layer="95"/>
 </segment>
 </net>
@@
 <segment>
 <pinref part="TP4" gate="G$1" pin="TP"/>
-<wire x1="180.34" y1="45.72" x2="172.72" y2="45.72" width="0.1524" layer="91"/>
-<label x="172.72" y="45.72" size="1.778" layer="95"/>
+<wire x1="96.52" y1="40.64" x2="88.9" y2="40.64" width="0.1524" layer="91"/>
+<label x="88.9" y="40.64" size="1.778" layer="95"/>
 </segment>
 </net>
@@
 <segment>
 <pinref part="TP3" gate="G$1" pin="TP"/>
-<wire x1="180.34" y1="48.26" x2="172.72" y2="48.26" width="0.1524" layer="91"/>
-<label x="172.72" y="48.26" size="1.778" layer="95"/>
+<wire x1="96.52" y1="43.18" x2="88.9" y2="43.18" width="0.1524" layer="91"/>
+<label x="88.9" y="43.18" size="1.778" layer="95"/>
 </segment>
 </net>
@@
 </segment>
 </net>
-<net name="N$5" class="0">
-<segment>
-<pinref part="IC1" gate="G$1" pin="VDD"/>
-<wire x1="22.86" y1="45.72" x2="15.24" y2="45.72" width="0.1524" layer="91"/>
-<pinref part="C1" gate="G$1" pin="2"/>
-<wire x1="15.24" y1="45.72" x2="15.24" y2="46.99" width="0.1524" layer="91"/>
-</segment>
-</net>

Commit message: Add files via upload
Connections:
- net +3V3: now also R2.1
- net +5V: no longer R2.1
Changed lines of the file:
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@@
 <part name="GND4" library="supply1" library_urn="urn:adsk.eagle:library:371" deviceset="GND" device=""/>
 <part name="P+2" library="supply1" library_urn="urn:adsk.eagle:library:371" deviceset="+5V" device=""/>
-<part name="P+3" library="supply1" library_urn="urn:adsk.eagle:library:371" deviceset="+5V" device=""/>
 <part name="GND5" library="supply1" library_urn="urn:adsk.eagle:library:371" deviceset="GND" device=""/>
 <part name="U2" library="SparkFun-IC-Power" library_urn="urn:adsk.eagle:library:526" deviceset="V_REG_AP2112" device="K-3.3V" package3d_urn="urn:adsk.eagle:package:39060/1" value="3.3V"/>
@@
 <part name="C1" library="discretes-dev" deviceset="CAP0402" device="" value="100nf"/>
 <part name="+3V1" library="supply1" library_urn="urn:adsk.eagle:library:371" deviceset="+3V3" device=""/>
+<part name="+3V3" library="supply1" library_urn="urn:adsk.eagle:library:371" deviceset="+3V3" device=""/>
 </parts>
 <sheets>
@@
 <attribute name="VALUE" x="22.86" y="48.26" size="1.778" layer="96" rot="R180"/>
 </instance>
-<instance part="P+3" gate="1" x="78.74" y="53.34" smashed="yes" rot="R270">
-<attribute name="VALUE" x="73.66" y="55.88" size="1.778" layer="96"/>
-</instance>
 <instance part="GND5" gate="1" x="2.54" y="45.72" smashed="yes" rot="R270">
 <attribute name="VALUE" x="0" y="48.26" size="1.778" layer="96" rot="R270"/>
@@
 <instance part="+3V1" gate="G$1" x="15.24" y="60.96" smashed="yes">
 <attribute name="VALUE" x="12.7" y="55.88" size="1.778" layer="96" rot="R90"/>
+</instance>
+<instance part="+3V3" gate="G$1" x="78.74" y="53.34" smashed="yes" rot="R270">
+<attribute name="VALUE" x="73.66" y="55.88" size="1.778" layer="96"/>
 </instance>
 </instances>
@@
 </segment>
 <segment>
-<pinref part="P+3" gate="1" pin="+5V"/>
-<wire x1="73.66" y1="53.34" x2="76.2" y2="53.34" width="0.1524" layer="91"/>
-<pinref part="R2" gate="G$1" pin="1"/>
-</segment>
-<segment>
 <pinref part="P+2" gate="1" pin="+5V"/>
 <pinref part="IC1" gate="G$1" pin="VBUS"/>
@@
 <wire x1="137.16" y1="10.16" x2="137.16" y2="5.08" width="0.1524" layer="91"/>
 <label x="137.16" y="5.08" size="1.778" layer="95" rot="R90"/>
-</segment>
-</net>
-<net name="N$3" class="0">
-<segment>
-<pinref part="IC1" gate="G$1" pin="!RST"/>
-<wire x1="60.96" y1="53.34" x2="63.5" y2="53.34" width="0.1524" layer="91"/>
-<pinref part="R2" gate="G$1" pin="2"/>
 </segment>
 </net>
@@
 <junction x="15.24" y="53.34"/>
 </segment>
+<segment>
+<pinref part="R2" gate="G$1" pin="1"/>
+<pinref part="+3V3" gate="G$1" pin="+3V3"/>
+<wire x1="73.66" y1="53.34" x2="76.2" y2="53.34" width="0.1524" layer="91"/>
+</segment>
 </net>
 <net name="PB01" class="0">
@@
 </segment>
 </net>
+<net name="N$3" class="0">
+<segment>
+<pinref part="IC1" gate="G$1" pin="!RST"/>
+<pinref part="R2" gate="G$1" pin="2"/>
+<wire x1="60.96" y1="53.34" x2="63.5" y2="53.34" width="0.1524" layer="91"/>
+</segment>
+</net>

Commit message: Add files via upload
Parts:
- added C2: 100n, discretes-dev:CAP0402
Connections:
- net +3V3: now also C2.1
- net GND: now also C2.2
Changed lines of the file:
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@@
 <part name="+3V1" library="supply1" library_urn="urn:adsk.eagle:library:371" deviceset="+3V3" device=""/>
 <part name="+3V3" library="supply1" library_urn="urn:adsk.eagle:library:371" deviceset="+3V3" device=""/>
+<part name="C2" library="discretes-dev" deviceset="CAP0402" device="" value="100n"/>
+<part name="GND7" library="supply1" library_urn="urn:adsk.eagle:library:371" deviceset="GND" device=""/>
 </parts>
 <sheets>
@@
 <attribute name="VALUE" x="73.66" y="55.88" size="1.778" layer="96"/>
 </instance>
+<instance part="C2" gate="G$1" x="162.56" y="30.48" smashed="yes">
+<attribute name="NAME" x="164.084" y="32.131" size="1.778" layer="95" font="vector"/>
+</instance>
+<instance part="GND7" gate="1" x="162.56" y="22.86" smashed="yes">
+<attribute name="VALUE" x="160.02" y="20.32" size="1.778" layer="96"/>
+</instance>
 </instances>
 <busses>
@@
 <wire x1="6.35" y1="45.72" x2="5.08" y2="45.72" width="0.1524" layer="91"/>
 <pinref part="GND5" gate="1" pin="GND"/>
+</segment>
+<segment>
+<pinref part="C2" gate="G$1" pin="2"/>
+<pinref part="GND7" gate="1" pin="GND"/>
+<wire x1="162.56" y1="26.67" x2="162.56" y2="25.4" width="0.1524" layer="91"/>
 </segment>
 </net>
@@
 <segment>
 <pinref part="U$1" gate="G$1" pin="VCC"/>
-<wire x1="157.48" y1="35.56" x2="165.1" y2="35.56" width="0.1524" layer="91"/>
+<wire x1="157.48" y1="35.56" x2="162.56" y2="35.56" width="0.1524" layer="91"/>
 <label x="160.02" y="35.56" size="1.778" layer="95"/>
-</segment>
-<segment>
+<pinref part="C2" gate="G$1" pin="1"/>
+<wire x1="162.56" y1="35.56" x2="165.1" y2="35.56" width="0.1524" layer="91"/>
+<wire x1="162.56" y1="34.29" x2="162.56" y2="35.56" width="0.1524" layer="91"/>
+<junction x="162.56" y="35.56"/>
+</segment>
+<segment>

Commit message: Add files via upload
Parts:
- added R6, R7, R8: 10k, SparkFun-Resistors:RESISTOR0402
Connections:
- new net N$5: IC1.!SUSPEND, R6.2
- net GND: now also R6.1, R7.2, R8.2
- net PB00: now also R7.1
- net PB01: now also R8.1
Changed lines of the file:
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@@
 <part name="C2" library="discretes-dev" deviceset="CAP0402" device="" value="100n"/>
 <part name="GND7" library="supply1" library_urn="urn:adsk.eagle:library:371" deviceset="GND" device=""/>
+<part name="R6" library="SparkFun-Resistors" library_urn="urn:adsk.eagle:library:532" deviceset="RESISTOR" device="0402" package3d_urn="urn:adsk.eagle:package:39657/1" value="10k"/>
+<part name="GND8" library="supply1" library_urn="urn:adsk.eagle:library:371" deviceset="GND" device=""/>
+<part name="R7" library="SparkFun-Resistors" library_urn="urn:adsk.eagle:library:532" deviceset="RESISTOR" device="0402" package3d_urn="urn:adsk.eagle:package:39657/1" value="10k"/>
+<part name="R8" library="SparkFun-Resistors" library_urn="urn:adsk.eagle:library:532" deviceset="RESISTOR" device="0402" package3d_urn="urn:adsk.eagle:package:39657/1" value="10k"/>
+<part name="GND9" library="supply1" library_urn="urn:adsk.eagle:library:371" deviceset="GND" device=""/>
 </parts>
 <sheets>
@@
 <attribute name="VALUE" x="160.02" y="20.32" size="1.778" layer="96"/>
 </instance>
+<instance part="R6" gate="G$1" x="68.58" y="45.72" smashed="yes" rot="R180">
+<attribute name="NAME" x="68.58" y="44.196" size="1.778" layer="95" font="vector" rot="R180" align="bottom-center"/>
+</instance>
+<instance part="GND8" gate="1" x="76.2" y="40.64" smashed="yes">
+<attribute name="VALUE" x="73.66" y="38.1" size="1.778" layer="96"/>
+</instance>
+<instance part="R7" gate="G$1" x="71.12" y="15.24" smashed="yes" rot="R270">
+<attribute name="NAME" x="72.644" y="15.24" size="1.778" layer="95" font="vector" rot="R270" align="bottom-center"/>
+</instance>
+<instance part="R8" gate="G$1" x="66.04" y="15.24" smashed="yes" rot="R270">
+<attribute name="NAME" x="67.564" y="15.24" size="1.778" layer="95" font="vector" rot="R270" align="bottom-center"/>
+</instance>
+<instance part="GND9" gate="1" x="68.58" y="5.08" smashed="yes">
+<attribute name="VALUE" x="66.04" y="2.54" size="1.778" layer="96"/>
+</instance>
 </instances>
 <busses>
@@
 <pinref part="GND7" gate="1" pin="GND"/>
 <wire x1="162.56" y1="26.67" x2="162.56" y2="25.4" width="0.1524" layer="91"/>
+</segment>
+<segment>
+<pinref part="R6" gate="G$1" pin="1"/>
+<wire x1="73.66" y1="45.72" x2="76.2" y2="45.72" width="0.1524" layer="91"/>
+<pinref part="GND8" gate="1" pin="GND"/>
+<wire x1="76.2" y1="45.72" x2="76.2" y2="43.18" width="0.1524" layer="91"/>
+</segment>
+<segment>
+<pinref part="R8" gate="G$1" pin="2"/>
+<wire x1="66.04" y1="10.16" x2="66.04" y2="7.62" width="0.1524" layer="91"/>
+<wire x1="66.04" y1="7.62" x2="68.58" y2="7.62" width="0.1524" layer="91"/>
+<pinref part="R7" gate="G$1" pin="2"/>
+<wire x1="68.58" y1="7.62" x2="71.12" y2="7.62" width="0.1524" layer="91"/>
+<wire x1="71.12" y1="7.62" x2="71.12" y2="10.16" width="0.1524" layer="91"/>
+<pinref part="GND9" gate="1" pin="GND"/>
+<junction x="68.58" y="7.62"/>
 </segment>
 </net>
@@
 <segment>
 <pinref part="IC1" gate="G$1" pin="CTS"/>
-<wire x1="60.96" y1="22.86" x2="68.58" y2="22.86" width="0.1524" layer="91"/>
+<wire x1="60.96" y1="22.86" x2="66.04" y2="22.86" width="0.1524" layer="91"/>
 <label x="63.5" y="22.86" size="1.778" layer="95"/>
+<pinref part="R8" gate="G$1" pin="1"/>
+<wire x1="66.04" y1="22.86" x2="68.58" y2="22.86" width="0.1524" layer="91"/>
+<wire x1="66.04" y1="22.86" x2="66.04" y2="20.32" width="0.1524" layer="91"/>
+<junction x="66.04" y="22.86"/>
 </segment>
 </net>
@@
 <segment>
 <pinref part="IC1" gate="G$1" pin="RTS"/>
-<wire x1="60.96" y1="25.4" x2="68.58" y2="25.4" width="0.1524" layer="91"/>
-<label x="63.5" y="25.4" size="1.778" layer="95"/>
+<label x="68.58" y="25.4" size="1.778" layer="95"/>
+<wire x1="60.96" y1="25.4" x2="71.12" y2="25.4" width="0.1524" layer="91"/>
+<pinref part="R7" gate="G$1" pin="1"/>
+<wire x1="71.12" y1="25.4" x2="73.66" y2="25.4" width="0.1524" layer="91"/>
+<wire x1="71.12" y1="20.32" x2="71.12" y2="25.4" width="0.1524" layer="91"/>
+<junction x="71.12" y="25.4"/>
 </segment>
 </net>
@@
 </segment>
 </net>
+<net name="N$5" class="0">
+<segment>
+<pinref part="IC1" gate="G$1" pin="!SUSPEND"/>
+<pinref part="R6" gate="G$1" pin="2"/>
+<wire x1="60.96" y1="45.72" x2="63.5" y2="45.72" width="0.1524" layer="91"/>
+</segment>
+</net>
