File: USB-PCB-A/sc_v1.brd (EAGLE design)
At the start: 36.4 x 15.2 mm, 22 parts, among them IC1 CP2102, U2 3.3V

Commit message: Add files via upload
Parts:
- moved R4 1.43 mm to (20.3, 7.89)
- moved R3 1.33 mm to (20.4, 9.28)
- moved R2 0.51 mm to (15.7, 3.38)
- moved R6 0.50 mm to (15.7, 3.40)
- moved D4 0.36 mm to (17.2, 7.97), turned to 90 degrees
- moved C1 0.10 mm to (20.1, 6.50)
Routing:
- net N$2: track 8.84 -> 4.88 mm, vias 2 -> 0
- net D-: track 16.5 -> 13.4 mm, vias 2 -> 0
- net +5V: track 29.7 -> 28.9 mm, vias 2 -> 3
- net N$1: track 6.08 -> 6.85 mm
- net +3V3: track 37.5 -> 38.0 mm
- net N$5: track 2.32 -> 2.84 mm
- net GND: vias 22 -> 20
Other:
- board size 36.4 x 15.2 mm -> 36.5 x 15.2 mm

Commit message: Add files via upload
Parts:
- removed C2: 100n, discretes-dev:CAPC1005X40N
- moved R8 13.4 mm to (22.8, 14.1), flipped to the top, turned to 180 degrees
- moved R7 11.0 mm to (22.2, 11.4), flipped to the top
- moved R6 7.99 mm to (23.3, 0.90), flipped to the top, turned to 0 degrees
- moved IC1 0.13 mm to (19.3, 2.64)
Connections:
- net +3V3: no longer C2.1
- net GND: no longer C2.2
Routing:
- net PB00: track 22.1 -> 34.7 mm, vias 1 -> 2
- net PB01: track 22.6 -> 34.0 mm, vias 1 -> 2
- net N$5: track 2.84 -> 11.7 mm, vias 1 -> 2
- net +3V3: track 38.0 -> 35.8 mm, vias 5 -> 4
- net +5V: track 28.9 -> 27.4 mm
- net D-: track 13.4 -> 14.1 mm
- net D+: track 13.4 -> 14.0 mm
- net GND: track 13.5 -> 14.1 mm, vias 20 -> 18
