File: USB-PCB-A/sc_v1.sch (EAGLE design)
At the start: 22 parts, among them IC1 CP2102, U2 3.3V

Commit message: Add files via upload
Parts:
- removed C2: 100n, discretes-dev:CAP0402
Connections:
- net +3V3: no longer C2.1
- net GND: no longer C2.2
Changed lines of the file:
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@@
 <part name="+3V1" library="supply1" library_urn="urn:adsk.eagle:library:371" deviceset="+3V3" device=""/>
 <part name="+3V3" library="supply1" library_urn="urn:adsk.eagle:library:371" deviceset="+3V3" device=""/>
-<part name="C2" library="discretes-dev" deviceset="CAP0402" device="" value="100n"/>
-<part name="GND7" library="supply1" library_urn="urn:adsk.eagle:library:371" deviceset="GND" device=""/>
 <part name="R6" library="SparkFun-Resistors" library_urn="urn:adsk.eagle:library:532" deviceset="RESISTOR" device="0402" package3d_urn="urn:adsk.eagle:package:39657/1" value="10k"/>
 <part name="GND8" library="supply1" library_urn="urn:adsk.eagle:library:371" deviceset="GND" device=""/>
@@
 <attribute name="VALUE" x="73.66" y="55.88" size="1.778" layer="96"/>
 </instance>
-<instance part="C2" gate="G$1" x="162.56" y="30.48" smashed="yes">
-<attribute name="NAME" x="164.084" y="32.131" size="1.778" layer="95" font="vector"/>
-</instance>
-<instance part="GND7" gate="1" x="162.56" y="22.86" smashed="yes">
-<attribute name="VALUE" x="160.02" y="20.32" size="1.778" layer="96"/>
-</instance>
 <instance part="R6" gate="G$1" x="68.58" y="45.72" smashed="yes" rot="R180">
 <attribute name="NAME" x="68.58" y="44.196" size="1.778" layer="95" font="vector" rot="R180" align="bottom-center"/>
@@
 <wire x1="6.35" y1="45.72" x2="5.08" y2="45.72" width="0.1524" layer="91"/>
 <pinref part="GND5" gate="1" pin="GND"/>
-</segment>
-<segment>
-<pinref part="C2" gate="G$1" pin="2"/>
-<pinref part="GND7" gate="1" pin="GND"/>
-<wire x1="162.56" y1="26.67" x2="162.56" y2="25.4" width="0.1524" layer="91"/>
 </segment>
 <segment>
@@
 <segment>
 <pinref part="U$1" gate="G$1" pin="VCC"/>
-<wire x1="157.48" y1="35.56" x2="162.56" y2="35.56" width="0.1524" layer="91"/>
+<wire x1="157.48" y1="35.56" x2="165.1" y2="35.56" width="0.1524" layer="91"/>
 <label x="160.02" y="35.56" size="1.778" layer="95"/>
-<pinref part="C2" gate="G$1" pin="1"/>
-<wire x1="162.56" y1="35.56" x2="165.1" y2="35.56" width="0.1524" layer="91"/>
-<wire x1="162.56" y1="34.29" x2="162.56" y2="35.56" width="0.1524" layer="91"/>
-<junction x="162.56" y="35.56"/>
-</segment>
-<segment>
+</segment>
+<segment>
