File: USB-A/sc_v1.brd (EAGLE design)
At the start: 29.2 x 15.2 mm, 21 parts, among them IC1 CP2102, J2 USB_A_SMT_MALE, U2 3.3V

Commit message: Add files via upload
Parts:
- moved J2 8.03 mm to (10.3, 9.90)
- moved TP7 7.84 mm to (43.8, 3.17)
- moved C3 7.84 mm to (23.7, 14.3)
- moved C4 7.84 mm to (26.8, 16.6)
- moved R6 7.84 mm to (30.7, 3.50)
- moved R7 7.84 mm to (29.6, 14.0)
- moved TP1 7.84 mm to (36.2, 3.17)
- moved TP2 7.84 mm to (37.4, 3.17)
- moved TP3 7.84 mm to (38.7, 3.15)
- moved C1 7.84 mm to (27.5, 9.10)
- moved D4 7.84 mm to (24.6, 10.6)
- moved IC1 7.84 mm to (26.7, 5.24)
- moved R3 7.84 mm to (27.8, 11.9)
- moved R4 7.84 mm to (27.7, 10.5)
- moved R8 7.84 mm to (30.2, 16.7)
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Routing:
- net GND: track 15.5 -> 4.76 mm, vias 18 -> 17
- net +3V3: track 35.8 -> 38.4 mm, vias 4 -> 5
- net N$3: track 1.37 -> 3.03 mm
- net +5V: track 21.4 -> 19.9 mm
Other:
- outline, holes or cut-outs redrawn

Commit message: Add files via upload
Parts:
- moved R6 15.8 mm to (21.7, 16.4)
- moved TP7 14.0 mm to (38.8, 16.3), flipped to the top
- moved TP1 13.6 mm to (32.5, 16.3), flipped to the top
- moved TP2 13.6 mm to (33.7, 16.3), flipped to the top
- moved TP3 13.6 mm to (35.0, 16.3), flipped to the top
- moved TP4 13.6 mm to (36.3, 16.3), flipped to the top
- moved TP5 13.6 mm to (37.6, 16.3), flipped to the top
- moved U$1 13.4 mm to (28.0, 3.47), flipped to the bottom, turned to 90 degrees
- moved R8 13.4 mm to (38.9, 6.50), turned to 90 degrees
- moved TP6 13.3 mm to (40.1, 16.3), flipped to the top
- moved R7 10.9 mm to (37.5, 6.50), turned to 90 degrees
- moved C4 3.78 mm to (29.8, 14.3), turned to 90 degrees
- moved C1 0.08 mm to (27.5, 9.18)
- moved IC1 0.08 mm to (26.7, 5.32)
Routing:
- net PB00: track 34.7 -> 11.2 mm, vias 2 -> 1
- net PB01: track 34.0 -> 13.1 mm, vias 2 -> 1
- net RX: track 14.5 -> 4.11 mm, vias 0 -> 1
- net +3V3: track 38.4 -> 31.5 mm, vias 5 -> 3
- net N$5: track 11.7 -> 16.1 mm
- net +5V: track 19.9 -> 23.9 mm
- net TDI: track 21.0 -> 17.8 mm
- net TCK: track 16.8 -> 14.8 mm
- net TX: track 7.19 -> 8.88 mm, vias 0 -> 1
- net TMS: track 17.7 -> 16.1 mm
- net RST: track 4.01 -> 3.29 mm
- net TDO: track 17.3 -> 16.7 mm
- net GND: track 4.76 -> 4.90 mm, vias 17 -> 20
Other:
- board size 29.2 x 15.2 mm -> 25.7 x 15 mm

Commit message: Add files via upload
Parts:
- moved R6 12.3 mm to (22.3, 4.13), flipped to the bottom, turned to 90 degrees
- moved C1 7.24 mm to (26.8, 16.4), turned to 0 degrees
- moved R3 4.04 mm to (24.4, 9.64), flipped to the bottom, turned to 0 degrees
- moved R4 3.41 mm to (24.4, 11.1), flipped to the bottom, turned to 0 degrees
- moved D4 1.32 mm to (23.4, 10.0), turned to 270 degrees
- flipped J2 to the bottom, turned to 180 degrees
Routing:
- net N$5: track 16.1 -> 2.43 mm, vias 2 -> 1
- net D-: track 8.06 -> 5.13 mm, vias 0 -> 1
- net +5V: track 23.9 -> 26.8 mm, vias 3 -> 1
- net D+: track 7.46 -> 5.76 mm, vias 0 -> 1
- net N$1: track 7.12 -> 5.72 mm, vias 0 -> 1
- net +3V3: track 31.5 -> 30.2 mm
- net N$2: track 5.04 -> 4.53 mm, vias 0 -> 1
